Commit message: Included Kinect RGBD sensor

File: eufs_description/robots/ads-dv.urdf.xacro (robot description, xacro)
@@ -58,7 +58,10 @@
         <origin xyz="1.58 0.0 -0.1" rpy="0 0 0" />
     </xacro:VLP-16R>
-    <xacro:zed_camera parent="base_link" prefix="zed">
+    <!-- <xacro:zed_camera parent="base_link" prefix="zed">
         <origin xyz="0.1 0.0 0.52" rpy="0 0 0" />
-    </xacro:zed_camera>
+    </xacro:zed_camera> -->
+    <xacro:sensor_kinect parent="base_link" prefix="kinect">
+        <origin xyz="0.0 0.0 0.45" rpy="0 0 0"/>
+    </xacro:sensor_kinect>
     <!-- EXTRA SENSORS FROM THE ROBOTNIK SENSORS LIBRARY -->
     <!--
